File: semana2/ejercicio2/ejercicio2/ejercicio2.kicad_sch (KiCad schematic)
At the start: 2 parts, among them U2 DHT11

Commit message: update all weeks
correccion de redaccion
Parts:
- removed U1: ~, ESP32_30pin, symbol esp32_30pin:ESP32_30Pin
- removed U2: DHT11, Sensor:Aosong_DHT11_5.5x12.0_P2.54mm, symbol Sensor:DHT11
